File: ESP32S3/ESP32S3.kicad_pcb (KiCad board)
At the start: 2 copper layers, 27.9 x 57.1 mm, 40 parts, among them IC1 RT9080N-08GJ5, J1 USB_C_Receptacle_USB2.0_16P, J2 Conn_01x18_Pin, J3 Conn_01x18_Pin, J4 USB_C_Receptacle_PowerOnly_6P, SW1 SW_MEC_5E, SW2 SW_MEC_5E, U1 ADUM3160, U2 ESP32-S3-WROOM-1, U3 CH340K, U4 TS5A23159DGS

Commit message: commit2605161301
Parts:
- removed U5: ~, footprints:SSAJ120100
- added C11: 0.1u, Capacitor_SMD:C_0603_1608Metric, B.Cu at (225.8, 97.6)
- added C12: 0.1u, Capacitor_SMD:C_0603_1608Metric, B.Cu at (205.4, 59.0)
- added IC2: TC7W74FU, Yamaha:TC7W53FUF, B.Cu at (222.4, 97.0)
- added Q1: BSS138, Package_TO_SOT_SMD:SOT-23, B.Cu at (209.8, 84.1)
- added Q2: BSS138, Package_TO_SOT_SMD:SOT-23, B.Cu at (214.3, 84.1)
- added R11: 24, Resistor_SMD:R_0603_1608Metric, F.Cu at (212.4, 89.5)
- added R12: 24, Resistor_SMD:R_0603_1608Metric, F.Cu at (212.4, 91.6)
- added R17: 10k, Resistor_SMD:R_0603_1608Metric_Pad0.98x0.95mm_HandSolder, B.Cu at (217.7, 95.2)
- added R3: 24, Resistor_SMD:R_0603_1608Metric, B.Cu at (210.4, 103.4)
- added R4: 24, Resistor_SMD:R_0603_1608Metric, B.Cu at (210.4, 105.0)
- added SW3: SW_MEC_5E, Yamaha:SW_SKRPABE010, F.Cu at (222.4, 96.6)
- C1: renamed from C3; value C_Small -> 1u
- C10, C9: value C_Small -> 0.1u
- C3: renamed from C1; value C_Small -> 1u
- C4: renamed from C7; value C_Small -> 1u
- C6: renamed from C2; value C_Small -> 1u
- C7: renamed from C4; value C_Small -> 1u
- C8: value C_Small -> 1u
- D4: renamed from D3; value WS2812B -> WS2812B5050
- moved R15 11.8 mm to (218.6, 97.8), turned to -90 degrees
- moved D3 10.5 mm to (218.6, 97.8), turned to -90 degrees
- moved D1 8.85 mm to (219.3, 101.2)
- moved R13 7.28 mm to (219.3, 101.2), turned to 180 degrees
- moved C2 5.76 mm to (222.1, 93.0), turned to 180 degrees
- moved R14 5.61 mm to (223.9, 101.2)
- moved C8 5.22 mm to (224.8, 104.0), turned to -90 degrees
- moved D2 4.19 mm to (223.9, 101.2), turned to 0 degrees
- moved C5 3.44 mm to (222.1, 90.0), turned to 180 degrees
- moved C6 1.63 mm to (209.1, 90.5), turned to 0 degrees
- moved R7 1.42 mm to (210.4, 101.8)
- moved U2 1.31 mm to (221.2, 92.0), turned to 0 degrees
- moved R8 1.07 mm to (210.4, 100.1)
- moved C4 1.03 mm to (218.4, 104.0), turned to 90 degrees
- moved IC1 0.90 mm to (221.6, 104.0), turned to 0 degrees
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- renumbered C5 to C2, C6 to C5, D4 to D3, J4 to J2, J2 to J4, R2 to R1, R7 to R10, R8 to R13, R9 to R14, R12 to R15, R1 to R16, R3 to R2, R10 to R5, R11 to R6, R5 to R7, R6 to R8, R4 to R9, U4 to U1, U3 to U2, U1 to U3, U2 to U4
Connections:
- C10 pad 2: DTR# -> IO0
- J1 pad A6: Net-(JP2-A) -> Net-(J1-D+-PadA6)
- J1 pad A7: Net-(JP1-A) -> Net-(J1-D--PadA7)
- J1 pad B6: Net-(JP2-A) -> Net-(J1-D+-PadA6)
- J1 pad B7: Net-(JP1-A) -> Net-(J1-D--PadA7)
- J4 pad 13: DTR# -> IO0
- JP1 pad 2: DD- -> d-
- JP2 pad 2: DD+ -> d+
- R15 pad 1: sw -> ~{sw}
- SW2 pad 1: DTR# -> IO0
- SW2 pad 2: DTR# -> IO0
- U2 pad 6: EN -> RTS#
- U3 pad 10: DD+ -> d+
- U3 pad 11: DD- -> d-
- U4 pad 27: DTR# -> IO0
Routing:
- net +5V: track 45.0 -> 4.90 mm
- net IO0: track 0.00 -> 35.4 mm, vias 0 -> 4
- net DTR#: track 55.2 -> 21.4 mm, vias 3 -> 2
- net RTS#: track 0.00 -> 27.4 mm, vias 0 -> 2
- net sw: track 38.2 -> 12.2 mm, vias 2 -> 0
- net EN: track 48.3 -> 31.2 mm, vias 2 -> 3
- net DD+: track 10.9 -> 0.83 mm
- net ck: track 0.00 -> 9.86 mm, vias 0 -> 1
- net d+: track 0.00 -> 9.63 mm
- net Net-(JP1-A): track 15.3 -> 6.73 mm, vias 2 -> 1
- net UD-: track 11.7 -> 3.36 mm
- net DD-: track 8.62 -> 0.82 mm
- net Net-(J1-D--PadA7): track 0.00 -> 6.76 mm, vias 0 -> 1
- net d-: track 0.00 -> 6.65 mm
- net Net-(JP2-A): track 14.6 -> 8.67 mm, vias 2 -> 1
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- added copper zone on In2.Cu, net +3V3
- added copper zone on In1.Cu, net +5V
- removed copper zone on B.Cu, net +3V3
- removed copper zone on F.Cu, net +5V
Other:
- copper layers 2 -> 4
