File: ESP32S3/ESP32S3.kicad_sch (KiCad schematic)
At the start: 40 parts, among them IC1 RT9080N-08GJ5, J1 USB_C_Receptacle_USB2.0_16P, J2 Conn_01x18_Pin, J3 Conn_01x18_Pin, J4 USB_C_Receptacle_PowerOnly_6P, SW1 SW_MEC_5E, SW2 SW_MEC_5E, U1 ADUM3160, U2 ESP32-S3-WROOM-1, U3 CH340K, U4 TS5A23159DGS

Commit message: commit2605161301
Parts:
- removed U5: ~, footprints:SSAJ120100, symbol Yamaha:SSAJ120100
- added C11, C12: 0.1u, Capacitor_SMD:C_0603_1608Metric, symbol Device:C_Small
- added IC2: TC7W74FU, Yamaha:TC7W53FUF, symbol Yamaha:TC7W74FU
- added Q1, Q2: BSS138, Package_TO_SOT_SMD:SOT-23, symbol Transistor_FET:BSS138
- added R11, R12, R3, R4: 24, Resistor_SMD:R_0603_1608Metric, symbol Device:R_Small
- added R17: 10k, Resistor_SMD:R_0603_1608Metric_Pad0.98x0.95mm_HandSolder, symbol Device:R_Small
- added SW3: SW_MEC_5E, Yamaha:SW_SKRPABE010, symbol Switch:SW_MEC_5E
- C1: renamed from C3; value C_Small -> 1u
- C10, C9: value C_Small -> 0.1u
- C3: renamed from C1; value C_Small -> 1u
- C4: renamed from C7; value C_Small -> 1u
- C6: renamed from C2; value C_Small -> 1u
- C7: renamed from C4; value C_Small -> 1u
- C8: value C_Small -> 1u
- D4: renamed from D3; value WS2812B -> WS2812B5050
- renumbered C5 to C2, C6 to C5, D4 to D3, J4 to J2, J2 to J4, R2 to R1, R7 to R10, R8 to R13, R9 to R14, R12 to R15, R1 to R16, R3 to R2, R10 to R5, R11 to R6, R5 to R7, R6 to R8, R4 to R9, U4 to U1, U3 to U2, U1 to U3, U2 to U4
Connections:
- net +3V3: now also C12.2
- net +5V: now also IC2.6 (~{CLR}), IC2.7 (~{PR}), IC2.8 (VCC)
- net DD+: now also R11.2; no longer JP2.2 (B), U3.10 (DD+)
- net DD-: now also R12.2; no longer JP1.2 (B), U3.11 (DD-)
- net DTR#: now also Q1.1 (G), Q2.2 (S); no longer C10.2, J4.13 (Pin_13), SW2.1, SW2.2, U4.27 (IO0)
- net EN: now also Q1.3 (D); no longer U2.6 (~{RTS})
- net GND: now also C11.1, C12.1, IC2.4 (GND), R17.2, SW3.3 (K), SW3.4 (A)
- net sw: now also IC2.5 (Q), R17.1; no longer R15.1
- net at JP1.1 (A), U3.6 (UD-): now also R3.2; no longer J1.A7 (D-), J1.B7 (D-)
- net at J1.A6 (D+), J1.B6 (D+): now also R4.1; no longer JP2.1 (A), U3.7 (UD+)
- new net: JP2.1 (A), R4.2, U3.7 (UD+)
- new net: J1.A7 (D-), J1.B7 (D-), R3.1
- new net IO0: C10.2, J4.13 (Pin_13), Q2.3 (D), SW2.1, SW2.2, U4.27 (IO0)
- new net RTS#: Q1.2 (S), Q2.1 (G), U2.6 (~{RTS})
- new net ck: C11.2, IC2.1 (CK), SW3.1, SW3.2
- new net d+: JP2.2 (B), R11.1, U3.10 (DD+)
- new net d-: JP1.2 (B), R12.1, U3.11 (DD-)
- new net ~{sw}: IC2.2 (D), IC2.3 (~{Q}), R15.1
- no-connect marks 7 -> 5
Other:
- note added: "designed by Terraria"
- note removed: "Terraria"
- moved on the sheet: C1, JP1, JP2
