File: ymz771/ymz771.kicad_pcb (KiCad board)
At the start: 2 copper layers, 72 x 72 mm, 99 parts, among them IC1 CH221K, J1 Conn_01x04_Pin, J2 Conn_02x12_Counter_Clockwise, J3 Conn_01x08_Pin, J4 Conn_02x08_Counter_Clockwise, J5 Conn_01x04_Pin, J6 Conn_01x05_Pin, J7 USB_C_Receptacle_PowerOnly_6P, J8 Conn_01x10_Pin, SW1 SW_DIP_x04, Y1 Crystal

Commit message: commit2605161301
Parts:
- removed C1, C4: C_Small, Capacitor_SMD:C_0603_1608Metric
- removed G***: LOGO, kokenlogo:kokenlogo10mm
- removed IC1: CH221K, YMZ771:SOT95P280X120-6N
- removed J3: Conn_01x08_Pin, Connector_PinHeader_2.54mm:PinHeader_1x08_P2.54mm_Vertical
- removed J5: Conn_01x04_Pin, Connector_PinSocket_2.54mm:PinSocket_1x04_P2.54mm_Vertical
- removed J6: Conn_01x05_Pin, Connector_PinHeader_2.54mm:PinHeader_1x05_P2.54mm_Vertical
- removed R21, R22, R23, R24, R25, R26, R27, R28, R29, R30, R31, R32: 10k, Resistor_SMD:R_0603_1608Metric_Pad0.98x0.95mm_HandSolder
- removed R33: 1k, Resistor_SMD:R_0603_1608Metric_Pad0.98x0.95mm_HandSolder
- removed R34, R35: 5.1k, Resistor_SMD:R_0603_1608Metric_Pad0.98x0.95mm_HandSolder
- removed R36, R38, R39, R40, R41, R42, R43, R44, R45, R46, R47, R48, R49, R50: 100k, Resistor_SMD:R_0603_1608Metric_Pad0.98x0.95mm_HandSolder
- added C17: 4u7, Capacitor_SMD:C_0603_1608Metric, F.Cu at (122.5, 132.3)
- added C18: 0.1u, Capacitor_SMD:C_0603_1608Metric, F.Cu at (189.5, 90.0)
- added C19: 47u, Capacitor_SMD:C_0603_1608Metric, F.Cu at (190.2, 96.9)
- added C20: 2.2uF, Capacitor_SMD:C_0603_1608Metric, F.Cu at (190.2, 99.4)
- added C21: 0.1u, Capacitor_SMD:C_0603_1608Metric, F.Cu at (190.2, 101.9)
- added C22: 47u, Capacitor_SMD:C_0603_1608Metric, F.Cu at (190.2, 104.4)
- added C23: C_Small, Capacitor_SMD:C_0603_1608Metric, F.Cu at (183.4, 136.9)
- added C24: C_Small, Capacitor_SMD:C_0603_1608Metric, F.Cu at (183.4, 139.4)
- added C25: C_Small, Capacitor_SMD:C_0603_1608Metric, F.Cu at (183.4, 141.9)
- added C26: 20n, Capacitor_SMD:C_0603_1608Metric_Pad1.08x0.95mm_HandSolder, B.Cu at (136.5, 102.9)
- added C27: C_Small, Capacitor_SMD:C_0603_1608Metric, F.Cu at (183.4, 144.4)
- added C28: C_Small, Capacitor_SMD:C_0603_1608Metric, F.Cu at (129.1, 109.4)
- added C29: 20n, Capacitor_SMD:C_0603_1608Metric_Pad1.08x0.95mm_HandSolder, B.Cu at (142.2, 100.1)
- added C30: 20n, Capacitor_SMD:C_0603_1608Metric_Pad1.08x0.95mm_HandSolder, B.Cu at (142.2, 94.4)
- added C31: C_Small, Capacitor_SMD:C_0603_1608Metric, F.Cu at (226.6, 47.0)
- added C32: C_Small, Capacitor_SMD:C_0603_1608Metric, F.Cu at (224.3, 52.3)
- added C33: 10uF, Capacitor_SMD:C_1812_4532Metric, F.Cu at (144.4, 146.1)
- added C34: 10uF, Capacitor_SMD:C_1812_4532Metric, F.Cu at (144.4, 151.0)
- added C35: C_Small, Capacitor_SMD:C_0603_1608Metric, F.Cu at (183.4, 146.9)
- added D16: LED_Small, LED_SMD:LED_0603_1608Metric_Pad1.05x0.95mm_HandSolder, F.Cu at (120.0, 114.8)
- added D17: LED_Small, LED_SMD:LED_0603_1608Metric_Pad1.05x0.95mm_HandSolder, F.Cu at (121.5, 114.8)
- added D18: LED_Small, LED_SMD:LED_0603_1608Metric_Pad1.05x0.95mm_HandSolder, F.Cu at (123.0, 114.8)
- added D19: LED_Small, LED_SMD:LED_0603_1608Metric_Pad1.05x0.95mm_HandSolder, F.Cu at (124.4, 114.8)
- added J10: Conn_02x08_Counter_Clockwise, Connector_PinHeader_1.27mm:PinHeader_2x08_P1.27mm_Vertical_SMD, F.Cu at (105.0, 91.7)
- added J11: Conn_02x12_Counter_Clockwise, Connector_PinHeader_1.27mm:PinHeader_2x12_P1.27mm_Vertical_SMD, F.Cu at (125.5, 80.0)
- added J9: Conn_02x06_Counter_Clockwise, Connector_PinHeader_1.27mm:PinHeader_2x06_P1.27mm_Vertical_SMD, F.Cu at (111.2, 80.0)
- added Q1: NMOS, Package_TO_SOT_SMD:SOT-23, B.Cu at (154.0, 68.5)
- added Q2: NMOS, Package_TO_SOT_SMD:SOT-23, F.Cu at (187.9, 133.0)
- added Q3: NMOS, Package_TO_SOT_SMD:SOT-23, B.Cu at (134.8, 56.9)
- added Q4: NMOS, Package_TO_SOT_SMD:SOT-23, F.Cu at (179.1, 86.0)
- added R55: 10k, Resistor_SMD:R_0603_1608Metric, F.Cu at (230.8, 50.4)
- added R56: 10k, Resistor_SMD:R_0603_1608Metric, F.Cu at (229.9, 55.5)
- added R57: 100k, Resistor_SMD:R_0603_1608Metric_Pad0.98x0.95mm_HandSolder, F.Cu at (150.1, 152.0)
- added RN1: R_Pack04, Yamaha:MNR04M0ABJ, B.Cu at (119.2, 85.0)
- added RN10: R_Pack04, Yamaha:MNR04M0ABJ, F.Cu at (122.2, 111.6)
- added RN11: R_Pack04, Yamaha:MNR04M0ABJ, F.Cu at (128.9, 111.6)
- added RN12: R_Pack04, Yamaha:MNR04M0ABJ, F.Cu at (134.8, 111.6)
- added RN13: R_Pack04, Yamaha:MNR04M0ABJ, B.Cu at (115.8, 116.8)
- added RN14: R_Pack04, Yamaha:MNR04M0ABJ, B.Cu at (115.8, 113.8)
- added RN2: R_Pack04, Yamaha:MNR04M0ABJ, B.Cu at (122.3, 85.0)
- added RN3: R_Pack04, Yamaha:MNR04M0ABJ, B.Cu at (125.3, 85.0)
- added RN4: R_Pack04, Yamaha:MNR04M0ABJ, B.Cu at (128.3, 85.0)
- added RN5: R_Pack04, Yamaha:MNR04M0ABJ, B.Cu at (131.3, 85.0)
- added RN6: R_Pack04, Yamaha:MNR04M0ABJ, B.Cu at (134.3, 85.0)
- added RN7: R_Pack04, Yamaha:MNR04M0ABJ, B.Cu at (135.2, 113.3)
- added RN8: R_Pack04, Yamaha:MNR04M0ABJ, B.Cu at (135.2, 116.3)
- added RN9: R_Pack04, Yamaha:MNR04M0ABJ, F.Cu at (116.3, 111.5)
- added SW2: RotaryEncoder, Rotary_Encoder:RotaryEncoder_Bourns_Horizontal_PEC09-2xxxF-Nxxxx, F.Cu at (230.0, 96.5)
- added SW3: SW_MEC_5E, Yamaha:SW_SKRPABE010, F.Cu at (168.9, 84.9)
- added U10: ESP32-S3-WROOM-1, RF_Module:ESP32-S3-WROOM-1, F.Cu at (78.8, 143.3)
- added U10: ~, YMZ771:YMZ771-F, F.Cu at (125.5, 98.5)
- added U11: 74AHC541, Package_SO:SSOP-20_5.3x7.2mm_P0.65mm, B.Cu at (121.5, 114.7)
- added U12: 74AHC541, Package_SO:SSOP-20_5.3x7.2mm_P0.65mm, B.Cu at (129.8, 114.7)
- added U13: ~, Package_DIP:DIP-8_W7.62mm, F.Cu at (153.8, 99.5)
- added U14: ~, Package_DIP:DIP-8_W7.62mm, F.Cu at (153.8, 111.4)
- added U2: TXS0104EPW, Package_SO:TSSOP-14_4.4x5mm_P0.65mm, B.Cu at (122.4, 89.4)
- added U3: ~, Package_TO_SOT_SMD:TSOT-23-5_HandSoldering, F.Cu at (233.4, 141.0)
- added U4: CH340K, Package_SO:SSOP-10-1EP_3.9x4.9mm_P1mm_EP2.1x3.3mm, B.Cu at (111.4, 109.4)
- added U5: TXS0104EPW, Package_SO:TSSOP-14_4.4x5mm_P0.65mm, F.Cu at (142.8, 105.0)
- added U6: ~, YMZ771:OSL2051A-LR, F.Cu at (153.0, 85.7)
- added U7: 74HC595, Package_SO:TSSOP-16_4.4x5mm_P0.65mm, B.Cu at (143.0, 82.4)
- added U8: PCM5102A, Package_SO:TSSOP-20_4.4x6.5mm_P0.65mm, B.Cu at (147.8, 113.6)
- added U9: ATmega4809-A, Package_QFP:TQFP-48_7x7mm_P0.5mm, B.Cu at (125.5, 98.5)
- C10: value C_Polarized_Small -> 0.1uF; footprint Capacitor_THT:CP_Radial_D6.3mm_P2.50mm -> Capacitor_SMD:C_0603_1608Metric
- C11, C2: value C_Small -> 0.1uF
- C12, C3: value 20n -> 0.1uF; footprint Capacitor_SMD:C_0603_1608Metric_Pad1.08x0.95mm_HandSolder -> Capacitor_SMD:C_0603_1608Metric
- C13: value C_Small -> 0.1uF; moved to F.Cu
- C14: value 20n -> 2.2nF; footprint Capacitor_SMD:C_0603_1608Metric_Pad1.08x0.95mm_HandSolder -> Capacitor_SMD:C_0603_1608Metric; moved to F.Cu
- C15: value C_Polarized_Small -> 2.2nF; footprint Capacitor_THT:CP_Radial_D8.0mm_P3.50mm -> Capacitor_SMD:C_0603_1608Metric
- C16: value C_Polarized_Small -> 2.2uF; footprint Capacitor_THT:CP_Radial_D8.0mm_P3.50mm -> Capacitor_SMD:C_0603_1608Metric
- C5, C6: value C_Small -> 0.1u
- C7: value C_Polarized_Small -> 0u1; footprint Capacitor_THT:CP_Radial_D6.3mm_P2.50mm -> Capacitor_SMD:C_0603_1608Metric
- C8, C9: value C_Polarized_Small -> 47u; footprint Capacitor_THT:CP_Radial_D6.3mm_P2.50mm -> Capacitor_SMD:C_0603_1608Metric
- D1: value LED_Small -> LED; footprint LED_SMD:LED_0603_1608Metric_Pad1.05x0.95mm_HandSolder -> LED_SMD:LED_0603_1608Metric
- J1: value Conn_01x04_Pin -> YMZ771-F; footprint Connector_PinHeader_2.54mm:PinHeader_1x04_P2.54mm_Vertical -> Yamaha:QFP80P1880X2480X295-80N
- J2: value Conn_02x12_Counter_Clockwise -> Micro_SD_Card_Det2; footprint Connector_PinHeader_2.54mm:PinHeader_2x12_P2.54mm_Vertical -> Connector_Card:microSD_HC_Hirose_DM3AT-SF-PEJM5; moved to B.Cu
- J4: value Conn_02x08_Counter_Clockwise -> MJ-8435; footprint Connector_PinHeader_2.54mm:PinHeader_2x08_P2.54mm_Vertical -> YMZ771:MJ-8435
- J7: value USB_C_Receptacle_PowerOnly_6P -> USB_C_Receptacle_USB2.0_16P; footprint Connector_USB:USB_C_Receptacle_GCT_USB4125-xx-x_6P_TopMnt_Horizontal -> Connector_USB:USB_C_Receptacle_GCT_USB4105-xx-A_16P_TopMnt_Horizontal
- J8: value Conn_01x10_Pin -> Conn_01x02_Pin; footprint Connector_PinHeader_2.54mm:PinHeader_1x10_P2.54mm_Vertical -> Connector_PinHeader_2.54mm:PinHeader_1x02_P2.54mm_Vertical
- R1: value 10k -> 5k1; footprint Resistor_SMD:R_0603_1608Metric_Pad0.98x0.95mm_HandSolder -> Resistor_SMD:R_0603_1608Metric
- R10, R13, R14, R15, R16, R6, R7, R8: value 10k -> R_Small; footprint Resistor_SMD:R_0603_1608Metric_Pad0.98x0.95mm_HandSolder -> Resistor_SMD:R_0603_1608Metric; moved to B.Cu
- R11, R17, R18, R19, R20, R5: footprint Resistor_SMD:R_0603_1608Metric_Pad0.98x0.95mm_HandSolder -> Resistor_SMD:R_0603_1608Metric
- R12, R9: value 10k -> 470; footprint Resistor_SMD:R_0603_1608Metric_Pad0.98x0.95mm_HandSolder -> Resistor_SMD:R_0603_1608Metric
- R2: value 10k -> 20k; footprint Resistor_SMD:R_0603_1608Metric_Pad0.98x0.95mm_HandSolder -> Resistor_SMD:R_0603_1608Metric
- R3, R4: value 10k -> 5k1; footprint Resistor_SMD:R_0603_1608Metric_Pad0.98x0.95mm_HandSolder -> Resistor_SMD:R_0603_1608Metric; moved to B.Cu
- R37: value 10k -> 100k; moved to F.Cu
- R51: value 100k -> 1M; footprint Resistor_SMD:R_0603_1608Metric_Pad0.98x0.95mm_HandSolder -> Resistor_SMD:R_0603_1608Metric
- SW1: value SW_DIP_x04 -> SW_Push; footprint Button_Switch_SMD:SW_DIP_SPSTx04_Slide_KingTek_DSHP04TS_W7.62mm_P1.27mm -> footprints:SKRPABE010
- U1: value ~ -> TS5A23159DGS; footprint YMZ771:YMZ771-F -> Package_SO:VSSOP-10_3x3mm_P0.5mm; moved to B.Cu
- Y1: value Crystal -> 16.384MHz; footprint Crystal:Crystal_SMD_HC49-SD -> Crystal:Crystal_SMD_3225-4Pin_3.2x2.5mm
- moved SW1 133.6 mm to (244.8, 131.2), turned to 0 degrees
- moved R37 114.2 mm to (211.9, 136.0)
- moved C5 111.9 mm to (235.4, 145.0), turned to 0 degrees
- moved J1 110.4 mm to (65.0, 171.0), turned to 0 degrees
- moved R11 92.4 mm to (229.0, 111.0), turned to 0 degrees
- moved C6 90.7 mm to (232.7, 149.7), turned to 0 degrees
- moved C13 82.3 mm to (189.4, 114.7), turned to 0 degrees
- moved C9 82.3 mm to (186.2, 99.4), turned to 0 degrees
- moved R5 81.3 mm to (205.2, 108.3), turned to 0 degrees
- moved C8 76.1 mm to (186.2, 96.9), turned to 0 degrees
- moved J4 70.6 mm to (175.8, 107.0), turned to -90 degrees
- moved C10 67.7 mm to (183.4, 131.8), turned to 0 degrees
- moved C11 66.0 mm to (183.4, 134.4), turned to 0 degrees
- moved R18 63.8 mm to (212.8, 114.9), turned to 0 degrees
- moved R1 56.4 mm to (176.0, 97.6), turned to 0 degrees
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Connections:
- C10 pad 1: AVDD -> +5V
- C11 pad 1: VDD4 -> GND
- C11 pad 2: GND -> +3V3
- C12 pad 1: Net-(U1-XO) -> +3V3
- C13 pad 1: Net-(IC1-VDD) -> +3V3
- C14 pad 1: /Vref -> GND
- C14 pad 2: GND -> OUTL
- C15 pad 1: /AOL -> GND
- C15 pad 2: Net-(J1-Pin_1) -> OUTR
- C16 pad 1: /AOR -> Net-(U8-CAPP)
- C16 pad 2: Net-(J1-Pin_3) -> Net-(U8-CAPM)
- C2 pad 1: AVDD -> GND
- C2 pad 2: GND -> +3V3
- C3 pad 1: Net-(U1-XI) -> GND
- C3 pad 2: GND -> +5V
- C5 pad 1: VDD2 -> GND
- C5 pad 2: GND -> +5V
- C6 pad 1: VDD4 -> GND
- C6 pad 2: GND -> +3V3
- C7 pad 1: VDD1 -> GND
- C7 pad 2: GND -> Net-(U4-V3)
- C8 pad 1: VDD2 -> GND
- C8 pad 2: GND -> +3V3
- C9 pad 1: VDD4 -> GND
- C9 pad 2: GND -> +3V3
- D1 pad 2: Net-(D1-A) -> TNOW
- D10 pad 1: GND -> Net-(D10-K)
- D11 pad 1: GND -> Net-(D11-K)
- D12 pad 1: GND -> Net-(D12-K)
- D13 pad 1: GND -> Net-(D13-K)
- D14 pad 1: GND -> Net-(D14-K)
- D15 pad 1: GND -> Net-(D15-K)
- D2 pad 1: GND -> Net-(D2-K)
- D2 pad 2: Net-(D2-A) -> +5V
- D4 pad 1: GND -> Net-(D4-K)
- D5 pad 1: GND -> Net-(D5-K)
- D6 pad 1: GND -> Net-(D6-K)
- D7 pad 1: GND -> Net-(D7-K)
- D8 pad 1: GND -> Net-(D8-K)
- D9 pad 1: GND -> Net-(D9-K)
- J1 pad 1: Net-(J1-Pin_1) -> /MD02
- J1 pad 2: GND -> /MD01
- J1 pad 3: Net-(J1-Pin_3) -> /MD00
- J1 pad 4: GND -> PC0
- J2 pad 1: /MA00 -> unconnected-(J2-DAT2-Pad1)
- J2 pad 10: /MA09 -> unconnected-(J2-DET_A-Pad10)
- J2 pad 11: /MA10 -> GND
- J2 pad 2: /MA01 -> Net-(J2-DAT3/CD)
- J2 pad 3: /MA02 -> Net-(J2-CMD)
- J2 pad 4: /MA03 -> +3V3
- J2 pad 5: /MA04 -> Net-(J2-CLK)
- J2 pad 6: /MA05 -> GND
- J2 pad 7: /MA06 -> Net-(J2-DAT0)
- J2 pad 8: /MA07 -> unconnected-(J2-DAT1-Pad8)
- J2 pad 9: /MA08 -> unconnected-(J2-DET_B-Pad9)
- J4 pad 1: /MD00 -> Net-(J4-Pad1)
- J4 pad 2: /MD01 -> GND
- J4 pad 3: /MD02 -> GND
- J4 pad 4: /MD03 -> Net-(J4-3)
- J7 pad A5: Net-(IC1-CC1) -> Net-(J7-CC1)
- J7 pad B5: Net-(IC1-CC2) -> Net-(J7-CC2)
- J8 pad 1: /AD -> +5V
- J8 pad 2: /ENA -> GND
- R1 pad 1: /MA00 -> +5V
- R1 pad 2: GND -> SP
- R10 pad 1: /MA09 -> Net-(U7-QD)
- R10 pad 2: GND -> Net-(U6-D)
- R11 pad 1: /MA10 -> Net-(Q1-D)
- R11 pad 2: GND -> +5V
- R12 pad 1: /MA11 -> OUTR
- R12 pad 2: GND -> Net-(U8-OUTR)
- R13 pad 1: /MA12 -> Net-(U7-QE)
- R13 pad 2: GND -> Net-(U6-E)
- R14 pad 1: /MA13 -> Net-(U7-QF)
- R14 pad 2: GND -> Net-(U6-F)
- R15 pad 1: /MA14 -> Net-(U7-QG)
- R15 pad 2: GND -> Net-(U6-G)
- R16 pad 1: /MA15 -> Net-(U7-QH)
- R16 pad 2: GND -> Net-(U6-DP)
- R17 pad 1: /MA16 -> Net-(D1-K)
- R18 pad 1: /MA17 -> GND
- R18 pad 2: GND -> 7seg
- R19 pad 1: /MA18 -> /PLAY#
- R19 pad 2: GND -> +5V
- R2 pad 1: /MA01 -> Net-(U14-IN+)
- R20 pad 1: /MA19 -> Net-(Q4-S)
- R20 pad 2: GND -> +3V3
- R3 pad 1: /MA02 -> GND
- R3 pad 2: GND -> Net-(J7-CC1)
- R37 pad 1: Net-(IC1-CFG) -> Net-(D2-K)
- R37 pad 2: Net-(IC1-VDD) -> /PLAY#
- R4 pad 1: /MA03 -> Net-(J7-CC2)
- R5 pad 1: /MA04 -> Net-(Q1-G)
- R5 pad 2: GND -> 7seg
- R51 pad 1: Net-(D15-A) -> Net-(J1-XI)
- R51 pad 2: //CS -> Net-(J1-XO)
- R6 pad 1: /MA05 -> Net-(U7-QA)
- R6 pad 2: GND -> Net-(U6-A)
- R7 pad 1: /MA06 -> Net-(U7-QB)
- R7 pad 2: GND -> Net-(U6-B)
- R8 pad 1: /MA07 -> Net-(U7-QC)
- R8 pad 2: GND -> Net-(U6-C)
- R9 pad 1: /MA08 -> OUTL
- R9 pad 2: GND -> Net-(U8-OUTL)
- SW1 pad 1: +5V -> GND
- SW1 pad 2: +5V -> PF3
- SW1 pad 3: +5V -> (no net)
- SW1 pad 4: +5V -> (no net)
- U1 pad 1: /MD02 -> SP
- U1 pad 10: Net-(J3-Pin_7) -> SPL
- U1 pad 2: /MD01 -> OUTL
- U1 pad 3: /MD00 -> GND
- U1 pad 4: Net-(J3-Pin_1) -> OUTR
- U1 pad 5: Net-(J3-Pin_2) -> SP
- U1 pad 6: Net-(J3-Pin_3) -> SPR
- U1 pad 7: Net-(J3-Pin_4) -> AOR
- U1 pad 8: Net-(J3-Pin_5) -> +5V
- U1 pad 9: Net-(J3-Pin_6) -> AOL
- Y1 pad 1: Net-(U1-XI) -> Net-(J1-XI)
- Y1 pad 2: Net-(U1-XO) -> GND
Routing:
- net VDD4: track 109.1 -> 0.00 mm, vias 1 -> 0
- net VDD2: track 94.0 -> 0.00 mm, vias 2 -> 0
- net AVDD: track 88.8 -> 0.00 mm, vias 1 -> 0
- net VDD1: track 72.9 -> 0.00 mm, vias 2 -> 0
- net //PLAY: track 40.3 -> 0.00 mm, vias 1 -> 0
- net //RESET: track 39.1 -> 0.00 mm, vias 1 -> 0
- net /Vref: track 38.0 -> 0.00 mm, vias 1 -> 0
- net /MBMD: track 37.1 -> 0.00 mm, vias 1 -> 0
- net /SEL: track 35.2 -> 0.00 mm, vias 1 -> 0
- net /S6M: track 33.6 -> 0.00 mm, vias 1 -> 0
- net //CS: track 32.5 -> 0.00 mm, vias 1 -> 0
- net //WR: track 32.1 -> 0.00 mm, vias 1 -> 0
- net Net-(J3-Pin_8): track 32.0 -> 0.00 mm, vias 1 -> 0
- net /AD: track 32.0 -> 0.00 mm, vias 1 -> 0
- net /ENA: track 31.8 -> 0.00 mm, vias 1 -> 0
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- added copper zone on In2.Cu, net +3V3
- added copper zone on In1.Cu, net +5V
Other:
- board size 72 x 72 mm -> 72 x 47 mm
- copper layers 2 -> 4
- board text added: "GPIO"
- board text removed: "+ -"
- board text removed: "AOL"
- board text removed: "AOR"
- board text removed: "AVDD"
- board text removed: "BCO"
- board text removed: "CLKO"
- board text removed: "GND"
- board text removed: "LRO"
- board text removed: "MD00"
- board text removed: "SDO"
- board text removed: "VDD1"
- board text removed: "VDD2"
- board text removed: "VDD4"
- board text removed: "V_{REF}"
