File: ammeter2/ammeter2.kicad_pcb (KiCad board)
At the start: 4 copper layers, 25 x 15 mm, 46 parts, among them IC1 TMUXHS221NKGT, J1 USB_C_Receptacle_USB2.0_16P, J2 USB_C_Receptacle_USB2.0_16P, J3 USB_C_Receptacle_USB2.0_16P, SW1 SW_MEC_5E, SW2 SW_MEC_5E, U1 MCP1501-12xRW, U2 TLV9001IDCK, U3 INA181, U4 CH340E, U6 ATtiny1604-SS, U7 AP63203WU

Commit message: 2605171513
Routing:
- net VBUS: vias 7 -> 6
- net /ref: vias 6 -> 5

Commit message: 2605281137
Parts:
- removed IC1: TMUXHS221NKGT, Yamaha:TMUXHS221NKGT
- removed the R11 at (109.8, 55.3)
- removed the R12 at (109.9, 56.9)
- added C7: 0.1u, Yamaha:1005, F.Cu at (106.8, 56.0)
- added R13: 4.7k, Yamaha:R1005, F.Cu at (109.2, 54.8)
- added U6: TS5A23159DGS, Package_SO:TSSOP-10_3x3mm_P0.5mm, B.Cu at (108.6, 56.5)
- moved C6 5.02 mm to (112.8, 58.0), turned to 0 degrees
- moved R5 0.40 mm to (115.3, 63.7)
- renumbered C9 to C10, C10 to C11, C11 to C12, C16 to C13, C12 to C14, C13 to C15, C14 to C16, C15 to C17, C7 to C8, C8 to C9, R13 to R11, R14 to R12, R15 to R14, R16 to R15, U6 to U7, U7 to U8
Connections:
- U4 pad 10: +3V3 -> Net-(U4-V3)
Routing:
- net GND: track 13.0 -> 24.8 mm, vias 18 -> 36
- net /UPDI: track 2.45 -> 9.18 mm
- net /#RTS: track 6.69 -> 10.2 mm, vias 2 -> 3
- net Net-(R13-Pad1): track 0.00 -> 2.76 mm, vias 0 -> 1
- net Net-(R12-Pad1): track 12.4 -> 9.70 mm
- net Net-(R11-Pad1): track 10.2 -> 11.9 mm
- net Net-(U4-V3): track 0.00 -> 1.72 mm
- net /Tx: track 3.38 -> 4.71 mm
- net Net-(IC1-OEN): track 1.07 -> 0.00 mm
- net VBUS: track 4.77 -> 5.79 mm
- net Net-(IC1-DB+): track 0.96 -> 0.00 mm, vias 1 -> 0
- net /Rx: track 4.25 -> 5.17 mm
- net Net-(J1-CC1): track 17.9 -> 17.2 mm
- net /V0: track 4.56 -> 5.21 mm, vias 0 -> 2
- net Net-(J1-D--PadA7): track 19.5 -> 20.1 mm
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