File: ammeter2/ammeter2.kicad_sch (KiCad schematic)
At the start: 46 parts, among them IC1 TMUXHS221NKGT, J1 USB_C_Receptacle_USB2.0_16P, J2 USB_C_Receptacle_USB2.0_16P, J3 USB_C_Receptacle_USB2.0_16P, SW1 SW_MEC_5E, SW2 SW_MEC_5E, U1 MCP1501-12xRW, U2 TLV9001IDCK, U3 INA181, U4 CH340E, U6 ATtiny1604-SS, U7 AP63203WU

Commit message: 2605281137
Parts:
- removed IC1: TMUXHS221NKGT, Yamaha:TMUXHS221NKGT, symbol Yamaha:TMUXHS221NKGT
- removed R11: 4.7k, Yamaha:R1005, symbol Device:R_Small
- removed R12: 10k, Yamaha:R1005, symbol Device:R_Small
- added C7: 0.1u, Yamaha:1005, symbol Device:C_Small
- added R13: 4.7k, Yamaha:R1005, symbol Device:R_Small
- added U6: TS5A23159DGS, Package_SO:TSSOP-10_3x3mm_P0.5mm, symbol Analog_Switch:TS5A23159DGS
- renumbered C9 to C10, C10 to C11, C11 to C12, C16 to C13, C12 to C14, C13 to C15, C14 to C16, C15 to C17, C7 to C8, C8 to C9, R13 to R11, R14 to R12, R15 to R14, R16 to R15, U6 to U7, U7 to U8
Connections:
- net #RTS: now also U6.1, U6.5
- net +3V3: now also U6.8 (VCC); no longer U4.10 (V3)
- net GND: now also C7.2, U6.3 (GND)
- net Rx: now also U6.10
- net Tx: now also U6.6
- net UPDI: now also R13.2, U6.2
- net at R12.1: now also U6.7
- net at R11.1: now also U6.9
- new net: R13.1, U6.4
- new net: C7.1, U4.10 (V3)
Other:
- moved on the sheet: C10, C11, C12, C8, C9, R10, R11, R12, R7, R8, R9, U5
